File: rev2/pcb/kicad/iCE40UP5K_logic_analyzer_rev2.kicad_sch (KiCad schematic)
At the start: 170 parts, among them IC1 ICE40UP5K-SG48I, IC2 MIC5504-3.3YM5-TR, IC3 MIC5504-1.2YM5-TR, IC4 FT2232HL-TRAY, IC5 W25Q40CLSNIG, IC6 SN74LVC14ADBRE4, IC7 SN74LVC14ADBRE4, IC8 SN74LVC14ADBRE4, J1 USB B Female Connector, J2 61300611121, J3 61202021621, J4 61300821121, J5 61300821121, J6 61300311121, J7 61300621121, Q1 2N7002H6327XTSA2, Y1 830208214809

Commit message: layout sorted with power pours on L3 and silkscreen
Parts:
- J4, J5: footprint LIB_2x4_61300821121:J_Wurth_WR-PHD_61300821121 -> 8pin_header_2x4_61300821121:J_Wurth_WR-PHD_61300821121
- J6: footprint LIB_1x3_61300311121:J_Wurth_WR-PHD_61300311121 -> 8pin_header_2x4_61300821121:J_Wurth_WR-PHD_61300311121
- J7: footprint LIB_2x4_61300821121:J_Wurth_WR-PHD_61300621121 -> 6pin_header_2x3_61300621121:J_Wurth_WR-PHD_61300621121
- TP1: Silkscreen_text (none) -> TP:5V
- TP13: silkscreen_text (none) -> GND
- TP14: silkscreen_text GND -> TP:GND
- TP2: Silkscreen_text (none) -> TP:3V3
- TP3: Silkscreen_text (none) -> TP:1V2
- TP4: Silkscreen_text (none) -> GND
- TP5: Silkscreen_text (none) -> CDONE
- TP6: Silkscreen_text (none) -> CRST_B
- renumbered R68_unp1 to R68, TP15 to TP:1V2, TP10 to TP:1V8, TP26 to TP:1V8, TP29 to TP:3V3, TP11 to TP:3V3, TP22 to TP:3V3, TP12 to TP:3V3, TP21 to TP:GND, TP33 to TP:GND, TP27 to TP:GND, TP7 to TP:PWREN#, TP9 to TP:PWRSAV, TP24 to TP:REF, TP28 to TP:RESET#, TP8 to TP:SUSPEND#, TP18 to TP:VCCPLL, TP23 to TP:VPHY, TP25 to TP:VPLL
Other:
- note added: "DO NOT PLACE R68 (by default)"
Changed lines of the file:
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@@
 		)
 	)
+	(text "DO NOT PLACE R68\n(by default)"
+		(exclude_from_sim no)
+		(at 60.452 100.838 0)
+		(effects
+			(font
+				(size 1.27 1.27)
+			)
+		)
+	)
 	(text "INPUT AUXILIARIES\n- series resistors\n- weak pulldowns\n- Schmitt buffers"
 		(exclude_from_sim no)
@@
 		(on_board yes)
 		(dnp no)
-		(property "Reference" "TP21"
+		(property "Reference" "TP:GND"
 			(at 240.538 209.55 90)
 			(effects
@@
 			(project "iCE40UP5K_logic_analyzer_rev2"
 				(path "/84c66010-816c-4380-94a0-a9b9d431fb8c"
-					(reference "TP21")
+					(reference "TP:GND")
 					(unit 1)
 				)
@@
 			)
 		)
-		(property "Footprint" "LIB_1x3_61300311121:J_Wurth_WR-PHD_61300311121"
+		(property "Footprint" "8pin_header_2x4_61300821121:J_Wurth_WR-PHD_61300311121"
 			(at 13.97 217.17 0)
 			(effects
@@
 			)
 		)
-		(property "Datasheet" "https://www.we-online.com/en/components/products/datasheet/61300311121?ki"
+		(property "Datasheet" ""
 			(at 7.62 257.81 0)
 			(effects
@@
 			)
 		)
-		(property "Description" "2.54 mm THT Pin Header"
+		(property "Description" ""
 			(at 20.32 217.17 0)
 			(effects
@@
 		(on_board yes)
 		(dnp no)
-		(property "Reference" "TP15"
+		(property "Reference" "TP:1V2"
 			(at 367.792 29.21 90)
 			(effects
@@
 			(project "iCE40UP5K_logic_analyzer_rev2"
 				(path "/84c66010-816c-4380-94a0-a9b9d431fb8c"
-					(reference "TP15")
+					(reference "TP:1V2")
 					(unit 1)
 				)
@@
 			)
 		)
+		(property "silkscreen_text" "GND"
+			(at 48.26 214.63 0)
+			(effects
+				(font
+					(size 1.27 1.27)
+				)
+				(hide yes)
+			)
+		)
 		(pin "1"
 		)
@@
 		(on_board yes)
 		(dnp no)
-		(property "Reference" "TP28"
+		(property "Reference" "TP:RESET#"
 			(at 116.332 204.47 90)
 			(effects
@@
 			(project "iCE40UP5K_logic_analyzer_rev2"
 				(path "/84c66010-816c-4380-94a0-a9b9d431fb8c"
-					(reference "TP28")
+					(reference "TP:RESET#")
 					(unit 1)
 				)
@@
 			)
 		)
+		(property "Silkscreen_text" "TP:5V"
+			(at 83.82 210.82 0)
+			(effects
+				(font
+					(size 1.27 1.27)
+				)
+				(hide yes)
+			)
+		)
 		(pin "1"
 		)
@@
 		(on_board yes)
 		(dnp no)
-		(property "Reference" "TP24"
+		(property "Reference" "TP:REF"
 			(at 116.332 194.31 90)
 			(effects
@@
 			(project "iCE40UP5K_logic_analyzer_rev2"
 				(path "/84c66010-816c-4380-94a0-a9b9d431fb8c"
-					(reference "TP24")
+					(reference "TP:REF")
 					(unit 1)
 				)
@@
 			)
 		)
+		(property "Silkscreen_text" "GND"
+			(at 62.23 222.25 0)
+			(effects
+				(font
+					(size 1.27 1.27)
+				)
+				(hide yes)
+			)
+		)
 		(pin "1"
 		)
@@
 			)
 		)
+		(property "Silkscreen_text" "TP:3V3"
+			(at 95.25 213.36 0)
+			(effects
+				(font
+					(size 1.27 1.27)
+				)
+				(hide yes)
+			)
+		)
 		(pin "1"
 		)
@@
 		(on_board yes)
 		(dnp no)
-		(property "Reference" "R68_unp1"
+		(property "Reference" "R68"
 			(at 37.338 102.108 90)
 			(effects
@@
 			(project "iCE40UP5K_logic_analyzer_rev2"
 				(path "/84c66010-816c-4380-94a0-a9b9d431fb8c"
-					(reference "R68_unp1")
+					(reference "R68")
 					(unit 1)
 				)
@@
 		(on_board yes)
 		(dnp no)
-		(property "Reference" "TP8"
+		(property "Reference" "TP:SUSPEND#"
 			(at 205.74 268.986 90)
 			(effects
@@
 			(project "iCE40UP5K_logic_analyzer_rev2"
 				(path "/84c66010-816c-4380-94a0-a9b9d431fb8c"
-					(reference "TP8")
+					(reference "TP:SUSPEND#")
 					(unit 1)
 				)
@@
 			)
 		)
-		(property "Footprint" "LIB_2x4_61300821121:J_Wurth_WR-PHD_61300621121"
+		(property "Footprint" "6pin_header_2x3_61300621121:J_Wurth_WR-PHD_61300621121"
 			(at 87.63 213.36 0)
 			(effects
@@
 			)
 		)
-		(property "Datasheet" "https://www.we-online.com/en/components/products/datasheet/61300621121?ki"
+		(property "Datasheet" ""
 			(at 83.82 254 0)
 			(effects
@@
 			)
 		)
-		(property "Description" "2.54 mm THT Dual Pin Header"
+		(property "Description" ""
 			(at 71.12 213.36 0)
 			(effects
@@
 			)
 		)
+		(property "Silkscreen_text" "CRST_B"
+			(at 35.56 217.17 0)
+			(effects
+				(font
+					(size 1.27 1.27)
+				)
+				(hide yes)
+			)
+		)
 		(pin "1"
 		)
@@
 		(on_board yes)
 		(dnp no)
-		(property "Reference" "TP29"
+		(property "Reference" "TP:3V3"
 			(at 244.602 137.16 90)
 			(effects
@@
 			(project "iCE40UP5K_logic_analyzer_rev2"
 				(path "/84c66010-816c-4380-94a0-a9b9d431fb8c"
-					(reference "TP29")
+					(reference "TP:3V3")
 					(unit 1)
 				)
@@
 		(on_board yes)
 		(dnp no)
-		(property "Reference" "TP9"
+		(property "Reference" "TP:PWRSAV"
 			(at 225.552 168.91 90)
 			(effects
@@
 			(project "iCE40UP5K_logic_analyzer_rev2"
 				(path "/84c66010-816c-4380-94a0-a9b9d431fb8c"
-					(reference "TP9")
+					(reference "TP:PWRSAV")
 					(unit 1)
 				)
@@
 			)
 		)
-		(property "Footprint" "LIB_2x4_61300821121:J_Wurth_WR-PHD_61300821121"
+		(property "Footprint" "8pin_header_2x4_61300821121:J_Wurth_WR-PHD_61300821121"
 			(at 87.63 185.42 0)
 			(effects
@@
 		(on_board yes)
 		(dnp no)
-		(property "Reference" "TP11"
+		(property "Reference" "TP:3V3"
 			(at 300.482 22.86 90)
 			(effects
@@
 			(project "iCE40UP5K_logic_analyzer_rev2"
 				(path "/84c66010-816c-4380-94a0-a9b9d431fb8c"
-					(reference "TP11")
+					(reference "TP:3V3")
 					(unit 1)
 				)
@@
 		(on_board yes)
 		(dnp no)
-		(property "Reference" "TP18"
+		(property "Reference" "TP:VCCPLL"
 			(at 346.202 67.31 90)
 			(effects
@@
 			(project "iCE40UP5K_logic_analyzer_rev2"
 				(path "/84c66010-816c-4380-94a0-a9b9d431fb8c"
-					(reference "TP18")
+					(reference "TP:VCCPLL")
 					(unit 1)
 				)
@@
 			)
 		)
+		(property "Silkscreen_text" "TP:1V2"
+			(at 95.25 215.9 0)
+			(effects
+				(font
+					(size 1.27 1.27)
+				)
+				(hide yes)
+			)
+		)
 		(pin "1"
 		)
@@
 		(on_board yes)
 		(dnp no)
-		(property "Reference" "TP33"
+		(property "Reference" "TP:GND"
 			(at 238.76 264.922 0)
 			(effects
@@
 			(project "iCE40UP5K_logic_analyzer_rev2"
 				(path "/84c66010-816c-4380-94a0-a9b9d431fb8c"
-					(reference "TP33")
+					(reference "TP:GND")
 					(unit 1)
 				)
@@
 		(on_board yes)
 		(dnp no)
-		(property "Reference" "TP7"
+		(property "Reference" "TP:PWREN#"
 			(at 267.462 228.6 90)
 			(effects
@@
 			(project "iCE40UP5K_logic_analyzer_rev2"
 				(path "/84c66010-816c-4380-94a0-a9b9d431fb8c"
-					(reference "TP7")
+					(reference "TP:PWREN#")
 					(unit 1)
 				)
@@
 		(on_board yes)
 		(dnp no)
-		(property "Reference" "TP10"
+		(property "Reference" "TP:1V8"
 			(at 198.628 168.91 90)
 			(effects
@@
 			(project "iCE40UP5K_logic_analyzer_rev2"
 				(path "/84c66010-816c-4380-94a0-a9b9d431fb8c"
-					(reference "TP10")
+					(reference "TP:1V8")
 					(unit 1)
 				)
@@
 		(on_board yes)
 		(dnp no)
-		(property "Reference" "TP22"
+		(property "Reference" "TP:3V3"
 			(at 203.962 115.824 0)
 			(effects
@@
 			(project "iCE40UP5K_logic_analyzer_rev2"
 				(path "/84c66010-816c-4380-94a0-a9b9d431fb8c"
-					(reference "TP22")
+					(reference "TP:3V3")
 					(unit 1)
 				)
@@
 			)
 		)
-		(property "silkscreen_text" "GND"
+		(property "silkscreen_text" "TP:GND"
 			(at 279.4 36.83 90)
 			(effects
@@
 			)
 		)
-		(property "Footprint" "LIB_2x4_61300821121:J_Wurth_WR-PHD_61300821121"
+		(property "Footprint" "8pin_header_2x4_61300821121:J_Wurth_WR-PHD_61300821121"
 			(at 43.18 185.42 0)
 			(effects
@@
 			)
 		)
-		(property "Datasheet" "https://www.we-online.com/en/components/products/datasheet/61300821121?ki"
+		(property "Datasheet" ""
 			(at 39.37 226.06 0)
 			(effects
@@
 			)
 		)
-		(property "Description" "2.54 mm THT Dual Pin Header"
+		(property "Description" ""
 			(at 26.67 185.42 0)
 			(effects
@@
 		(on_board yes)
 		(dnp no)
-		(property "Reference" "TP25"
+		(property "Reference" "TP:VPLL"
 			(at 116.332 146.05 90)
 			(effects
@@
 			(project "iCE40UP5K_logic_analyzer_rev2"
 				(path "/84c66010-816c-4380-94a0-a9b9d431fb8c"
-					(reference "TP25")
+					(reference "TP:VPLL")
 					(unit 1)
 				)
@@
 		(on_board yes)
 		(dnp no)
-		(property "Reference" "TP23"
+		(property "Reference" "TP:VPHY"
 			(at 116.332 125.73 90)
 			(effects
@@
 			(project "iCE40UP5K_logic_analyzer_rev2"
 				(path "/84c66010-816c-4380-94a0-a9b9d431fb8c"
-					(reference "TP23")
+					(reference "TP:VPHY")
 					(unit 1)
 				)
@@
 		(on_board yes)
 		(dnp no)
-		(property "Reference" "TP26"
+		(property "Reference" "TP:1V8"
 			(at 193.802 137.16 90)
 			(effects
@@
 			(project "iCE40UP5K_logic_analyzer_rev2"
 				(path "/84c66010-816c-4380-94a0-a9b9d431fb8c"
-					(reference "TP26")
+					(reference "TP:1V8")
 					(unit 1)
 				)
@@
 		(on_board yes)
 		(dnp no)
-		(property "Reference" "TP12"
+		(property "Reference" "TP:3V3"
 			(at 198.628 179.07 90)
 			(effects
@@
 			(project "iCE40UP5K_logic_analyzer_rev2"
 				(path "/84c66010-816c-4380-94a0-a9b9d431fb8c"
-					(reference "TP12")
+					(reference "TP:3V3")
 					(unit 1)
 				)
@@
 		(on_board yes)
 		(dnp no)
-		(property "Reference" "TP27"
+		(property "Reference" "TP:GND"
 			(at 210.058 198.12 90)
 			(effects
@@
 			(project "iCE40UP5K_logic_analyzer_rev2"
 				(path "/84c66010-816c-4380-94a0-a9b9d431fb8c"
-					(reference "TP27")
+					(reference "TP:GND")
 					(unit 1)
 				)
@@
 			(at 35.56 219.71 0)
 			(effects
+				(font
+					(size 1.27 1.27)
+				)
+				(hide yes)
+			)
+		)
+		(property "Silkscreen_text" "CDONE"
+			(at 35.56 219.71 0)
+			(effects
