File: rev2/pcb/kicad/iCE40UP5K_logic_analyzer_rev2.kicad_pcb (KiCad board)
At the start: 4 copper layers, 89.7 x 82.9 mm, 170 parts, among them IC1 ICE40UP5K-SG48I, IC2 MIC5504-3.3YM5-TR, IC3 MIC5504-1.2YM5-TR, IC4 FT2232HL-TRAY, IC5 W25Q40CLSNIG, IC6 SN74LVC14ADBRE4, IC7 SN74LVC14ADBRE4, IC8 SN74LVC14ADBRE4, J1 USB B Female Connector, J2 61300611121, J3 61202021621, J4 61300821121, J5 61300821121, J6 61300311121, J7 61300621121, Q1 2N7002H6327XTSA2, Y1 830208214809

Commit message: PCB completed final DRC. Rev2 production files generated. PCB and components ordered.
Parts:
- moved J4 1.38 mm to (156.0, 141.8)
Routing:
- net /FPGA_DBG3: track 8.72 -> 10.1 mm
- net /FPGA_DBG2: track 8.72 -> 10.1 mm
- net /FPGA_DBG0: track 9.61 -> 11.0 mm
- net /FPGA_DBG1: track 9.67 -> 10.5 mm
Other:
- board text added: "."
- board text added: "DBG0"
- board text added: "DBG1"
- board text added: "DBG2"
- board text added: "DBG3"
- board text added: "External rail injection. One source only! (USB or EXT PWR)"
- board text added: "Logic Analyzer iCE40 UP5K Revision 2 11-07-2026 //JKO"
- board text removed: "DBG0..3"
- board text removed: "External rail injection for debugging only!"
- board text removed: "Logic Analyzer iCE40 UP5K Revision 2 10-07-2026 //JKO"
Changed lines of the file:
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@@
 			(sketchdnponfab yes)
 			(crossoutdnponfab yes)
-			(subtractmaskfromsilk no)
+			(subtractmaskfromsilk yes)
 			(outputformat 1)
 			(mirror no)
 			(drillshape 0)
 			(scaleselection 1)
-			(outputdirectory "gerbers/")
+			(outputdirectory "../production/gerbers/")
 		)
 	)
@@
 		(tags "test point SMD pad")
 		(property "Reference" "TP:VCCPLL"
-			(at 0 1.502174 0)
+			(at 2.4892 1.502174 0)
 			(layer "F.SilkS")
 			(effects
@@
 		)
 		(embedded_fonts no)
-		(model "150080YS75000.stp"
-			(offset
-				(xyz 0 0 0)
-			)
-			(scale
-				(xyz 1 1 1)
-			)
-			(rotate
-				(xyz 0 0 0)
-			)
-		)
 		(model "C:/Users/Jakob/Documents/Logic analyzer components KiCad/LIB_150080YS75000/150080YS75000/3D/150080YS75000.stp"
 			(offset
@@
 		)
 		(embedded_fonts no)
-		(model "APT2012LVBC_D.stp"
-			(offset
-				(xyz -0.02999999888 0 0.01999999925)
-			)
-			(scale
-				(xyz 1 1 1)
-			)
-			(rotate
-				(xyz -90 0 0)
-			)
-		)
 		(model "C:/Users/Jakob/Documents/Logic analyzer components KiCad/LIB_APT2012LVBC_D/APT2012LVBC_D/3D/APT2012LVBC_D.stp"
 			(offset
@@
 	(footprint "8pin_header_2x4_61300821121:J_Wurth_WR-PHD_61300821121"
 		(layer "F.Cu")
-		(at 155.9814 140.402 90)
+		(at 155.9814 141.7828 90)
 		(descr "2.54 mm THT Dual Pin Header, body 10.16x5.08x11.54mm, https://www.we-online.com/en/components/products/datasheet/61300821121?ki")
 		(tags "THT")
@@
 	)
 	(gr_text "GND"
-		(at 215.4174 97.2058 0)
+		(at 215.4174 97.265067 0)
 		(layer "F.SilkS")
 		(effects
@@
 	)
 	(gr_text "FPGA_DBG_HDR"
-		(at 165.5064 139.7254 0)
+		(at 165.5064 141.1062 0)
 		(layer "F.SilkS")
 		(effects
@@
 	)
 	(gr_text "FPGA_TX"
-		(at 202.870048 97.2566 0)
+		(at 202.870048 97.3074 0)
 		(layer "F.SilkS")
 		(effects
@@
 		)
 	)
-	(gr_text "DBG0..3"
-		(at 155.194 135.83 0)
+	(gr_text "DBG0"
+		(at 156.6164 137.3632 90)
 		(layer "F.SilkS")
 		(effects
@@
 		)
 	)
+	(gr_text "."
+		(at 136.327 130.7222 0)
+		(layer "F.SilkS")
+		(effects
+			(font
+				(size 1 0.8)
+				(thickness 0.16)
+			)
+		)
+	)
 	(gr_text "OFF"
 		(at 157.1244 67.5596 0)
@@
 		)
 	)
-	(gr_text "External rail injection\nfor debugging only!"
-		(at 211.1248 83.3628 0)
+	(gr_text "DBG3"
+		(at 164.2364 137.3632 90)
+		(layer "F.SilkS")
+		(effects
+			(font
+				(size 1 0.8)
+				(thickness 0.16)
+			)
+			(justify left bottom)
+		)
+	)
+	(gr_text "External rail injection.\nOne source only!\n(USB or EXT PWR)"
+		(at 211.1248 85.1662 0)
 		(layer "F.SilkS" knockout)
 		(effects
@@
 		)
 	)
+	(gr_text "DBG1"
+		(at 159.1564 137.3632 90)
+		(layer "F.SilkS")
+		(effects
+			(font
+				(size 1 0.8)
+				(thickness 0.16)
+			)
+			(justify left bottom)
+		)
+	)
 	(gr_text "GND"
 		(at 215.1634 75.565 0)
@@
 	)
 	(gr_text "GND"
-		(at 215.4174 99.6442 0)
+		(at 215.4174 99.822 0)
 		(layer "F.SilkS")
 		(effects
@@
 	)
 	(gr_text "CTS#"
-		(at 204.851 92.2782 0)
+		(at 204.851 92.1258 0)
 		(layer "F.SilkS")
 		(effects
@@
 	)
 	(gr_text "GND"
-		(at 215.4174 92.075 0)
+		(at 215.4174 92.1512 0)
 		(layer "F.SilkS")
 		(effects
@@
 	)
 	(gr_text "RTS#"
-		(at 204.851 94.7674 0)
+		(at 204.851 94.7166 0)
 		(layer "F.SilkS")
 		(effects
@@
 	)
 	(gr_text "FPGA_RX"
-		(at 202.679572 99.7458 0)
+		(at 202.679572 99.8982 0)
 		(layer "F.SilkS")
 		(effects
@@
 	)
 	(gr_text "GND"
-		(at 215.4174 94.7166 0)
+		(at 215.4174 94.708133 0)
 		(layer "F.SilkS")
 		(effects
@@
 	)
 	(gr_text "---GNDs---"
-		(at 155.3972 143.704 0)
+		(at 155.3972 145.0848 0)
 		(layer "F.SilkS")
 		(effects
@@
 	)
 	(gr_text "CONFIG_HDR"
-		(at 134.9248 135.763 0)
+		(at 134.7978 135.6614 0)
+		(layer "F.SilkS")
+		(effects
+			(font
+				(size 1 0.8)
+				(thickness 0.16)
+			)
+			(justify left bottom)
+		)
+	)
+	(gr_text "DBG2"
+		(at 161.6964 137.3632 90)
 		(layer "F.SilkS")
 		(effects
@@
 		)
 	)
-	(gr_text "Logic Analyzer\niCE40 UP5K\nRevision 2\n10-07-2026\n//JKO"
+	(gr_text "Logic Analyzer\niCE40 UP5K\nRevision 2\n11-07-2026\n//JKO"
 		(at 219.202 72.1868 0)
 		(layer "B.SilkS")
@@
 	)
 	(via
-		(at 217.3732 86.7664)
+		(at 217.3732 87.4268)
 		(size 0.7)
 		(drill 0.3)
@@
 	)
 	(via
-		(at 206.2226 86.7918)
+		(at 206.2226 87.4522)
 		(size 0.7)
 		(drill 0.3)
@@
 	)
 	(segment
-		(start 161.0614 137.862)
+		(start 161.5948 129.3612)
 		(end 161.0614 129.8946)
 		(width 0.2)
@@
 	(segment
 		(start 161.0614 129.8946)
-		(end 161.5948 129.3612)
+		(end 161.0614 139.2428)
 		(width 0.2)
 		(layer "F.Cu")
@@
 	)
 	(segment
-		(start 158.1658 137.5064)
-		(end 158.5214 137.862)
+		(start 158.5214 137.862)
+		(end 158.5214 139.2428)
 		(width 0.2)
 		(layer "F.Cu")
@@
 	)
 	(segment
+		(start 155.9814 137.862)
+		(end 155.9814 139.2428)
+		(width 0.2)
+		(layer "F.Cu")
+		(net 148)
+	)
+	(segment
 		(start 163.068 137.3286)
 		(end 163.6014 137.862)
@@
 	)
 	(segment
+		(start 163.6014 137.862)
+		(end 163.6014 139.2428)
+		(width 0.2)
+		(layer "F.Cu")
+		(net 149)
+	)
+	(segment
 		(start 162.8496 82.3876)
 		(end 162.8496 80.2732)
@@
 		(polygon
 			(pts
-				(xy 146.14 128.44) (xy 146.14 139.94) (xy 150.6 144.4) (xy 170.64 144.4) (xy 173.203549 141.836451)
+				(xy 146.14 128.44) (xy 146.14 139.94) (xy 151.362 145.162) (xy 169.878 145.162) (xy 173.203549 141.836451)
 				(xy 173.203549 135.03777) (xy 166.605779 128.44)
 			)
